File: TM4C-Red-Pill.kicad_sch (KiCad schematic)
At the start: 34 parts, among them IC1 TM4C123GH6PMI7R, J1 Conn_01x22, J2 Conn_01x22, J3 Conn_02x05_Odd_Even, J4 USB_C_Receptacle_USB2.0_16P, U1 TLV75533PDBV, U2 USBLC6-2SC6, Y1 ABM3-16.000MHZ-B2-T, Y2 ABS07-32.768KHZ-T

Commit message: Renamed project to TM4C Red Pill
Other:
- title: TM4C Purple Pill -> TM4C Red Pill
Changed lines of the file:
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@@
 	(paper "A4")
 	(title_block
-		(title "TM4C Purple Pill")
+		(title "TM4C Red Pill")
 		(date "2024-05-31")
 		(rev "0.3")
 		(company "Rolando Rosales")
-		(comment 1 "https://github.com/rolo-g/TM4C-Purple-Pill")
+		(comment 1 "https://github.com/rolo-g/TM4C-Red-Pill")
 	)
 	(junction
